File: hardware/pcb_files/air_node.brd (EAGLE design)
At the start: 124.5 x 58.4 mm, 31 parts, among them X1 RASPI_BOARD_B+#_E4

Commit message: pcb v0.2
added one-wire, uart, usb disconnector port and one more ads1115
Parts:
- added 1-WIRE: (no value), SparkFun-Connectors:1X03_NO_SILK
- added A0, A1, A2, A3, USB-DISCONNECTOR: (no value), SparkFun-Connectors:1X02_NO_SILK
- added C10, C11, C12, C13: (no value), rcl:C0805
- added LED_DISCO: (no value), led:CHIP-LED0805
- added R3, R4, R5, R6, R7, R8: (no value), rcl:R0805
- added U$7: ADC-4CH-ADS1115, diy-modules:ADC-4CH-ADS1115
- added UART: (no value), SparkFun-Connectors:1X04_NO_SILK
- moved SHT30 20.8 mm to (74.9, 72.4)
- moved J1 18.3 mm to (2.54, 25.7), turned to 270 degrees
Connections:
- removed net 3V3B: X1.17
- new net +3V3: 1-WIRE.1, R4.2, X1.17
- new net 1WIRE: 1-WIRE.2, R4.1, X1.36
- new net N$17: A1.1, C13.1, R7.1, U$7.8
- new net N$18: LED_DISCO.A, USB-DISCONNECTOR.2, X1.35
- new net N$19: A0.1, C12.1, R8.1, U$7.7
- new net N$20: A3.1, C10.1, R5.1, U$7.10
- new net N$21: A2.1, C11.1, R6.1, U$7.9
- new net N$22: LED_DISCO.C, R3.2
- new net RXD: UART.2, X1.10
- new net TXD: UART.3, X1.8
- net GND: now also 1-WIRE.3, A0.2, A1.2, A2.2, A3.2, C10.2, C11.2, C12.2, C13.2, R3.1, U$7.2, UART.4, USB-DISCONNECTOR.1
- net SCL1: now also U$7.3, U$7.5
- net SDA1: now also U$7.4
- net VCC/2: now also R5.2, R6.2, R7.2, R8.2, U$7.1, UART.1
Routing:
- net VCC/2: track 341.0 -> 512.0 mm
- net +3V3: track 0.00 -> 78.1 mm, vias 0 -> 2
- net N$19: track 0.00 -> 64.5 mm
- net N$17: track 0.00 -> 54.3 mm
- net SCL1: track 94.2 -> 147.7 mm
- net SDA1: track 105.6 -> 155.6 mm
- net N$21: track 0.00 -> 44.1 mm
- net 1WIRE: track 0.00 -> 41.3 mm
- net RXD: track 0.00 -> 37.8 mm, vias 0 -> 1
- net N$18: track 0.00 -> 37.5 mm
- net N$20: track 0.00 -> 33.9 mm
- net TXD: track 0.00 -> 33.0 mm, vias 0 -> 1
- net GND: track 25.0 -> 56.1 mm, vias 6 -> 7
- net 12VGND: track 27.6 -> 48.1 mm
- net N$22: track 0.00 -> 4.61 mm
Other:
- board size 124.5 x 58.4 mm -> 124.5 x 78.7 mm
- board text added: "air quality sensor node ver. 0.2"
- board text added: "data"
- board text added: "rxd"
- board text added: "txd"
- board text removed: "3-pin DC/DC is used"
- board text removed: "air quality sensor node ver. 0.1"
- board text removed: "only bridge J1 if small"
